File: ft4232h_mini_module.kicad_sch (KiCad schematic)
At the start: 22 parts, among them J1 Conn_01x20, J2 Conn_01x20, U1 74HC595, U2 FT4232H-56Q_MINI_MDL

Commit message: Update
Parts:
- D1, D2, D3, D4, D5, D6, D7, D8: value Red -> LED
- R1: value 10k -> 2.7k
- R2, R3, R4, R5, R6, R7, R8, R9: value 1.5k -> R
Other:
- note added: "LEDs & Resistors @ 10mcd Red (KP-2012SURC) = 2.2kΩ Green (KP-2012CGCK) = 330Ω Yellow (KP-2012SYCK) = 1kΩ"
- moved on the sheet: D1, D2, D3, D4, D5, D6, D7, D8, R2, R3, R4, R5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
